Commit message: change angles calculation

File: uarm_description/urdf/uarm.urdf.xacro (robot description, xacro)
@@ -32,5 +32,5 @@
     </link>
     <joint name="body_upper_arm_j" type="continuous">
-      <origin xyz="0.069 0 0.021" rpy="-${M_PI/2+0.624} 0 ${-M_PI/2}"/>
+      <origin xyz="0.069 0 0.021" rpy=-3 0 ${-M_PI/2}"/>
       <parent link="uarm_body_link"/>
       <child link="uarm_upper_arm_link"/>
@@ -46,5 +46,5 @@
     </link>
     <joint name="upper_arm_forearm_j" type="continuous">
-      <origin xyz="0 0.048 0.138 " rpy="${2.87} 0 0"/>
+      <origin xyz="0 0.048 0.138 " rpy="1.052 0 0"/>
       <parent link="uarm_upper_arm_link"/>
       <child link="uarm_forearm_link"/>
@@ -60,5 +60,5 @@
     </link>
     <joint name="forearm_wrist_j" type="continuous">
-      <origin xyz="0 -0.145 -0.068" rpy="${0.624-2.87} 0 0"/>
+      <origin xyz="0 -0.145 -0.068" rpy="-2.8 0 0"/>
       <parent link="uarm_forearm_link"/>
       <child link="uarm_wrist_link"/>

Commit message: added inverse kinematics angle calculation based on KDL library

File: uarm_description/urdf/uarm.urdf.xacro (robot description, xacro)
@@ -32,5 +32,5 @@
     </link>
     <joint name="body_upper_arm_j" type="continuous">
-      <origin xyz="0.069 0 0.021" rpy=-3 0 ${-M_PI/2}"/>
+      <origin xyz="0.069 0 0.021" rpy="-3 0 ${-M_PI/2}"/>
       <parent link="uarm_body_link"/>
       <child link="uarm_upper_arm_link"/>
