Commit message: workin with model

File: uarm_description/urdf/uarm3.urdf.xacro (robot description, xacro)
@@ -41,5 +41,5 @@
       <parent link="uarm_base_link"/>
       <child link="uarm_body_link"/>
-      <axis xyz="0 0 -1" />
+      <axis xyz="1 0 0" />
       <limit lower="${joint_lower_limit}" upper="${joint_upper_limit}" effort="${joint_effort}" velocity="${joint_velocity}" />
     </joint>
@@ -70,5 +70,5 @@
       <parent link="uarm_body_link"/>
       <child link="uarm_upper_arm_link"/>
-      <axis xyz="0 0 -1" />
+      <axis xyz="1 0 0" />
       <limit lower="${joint_lower_limit}" upper="${joint_upper_limit}" effort="${joint_effort}" velocity="${joint_velocity}" />
     </joint>
@@ -99,5 +99,5 @@
       <parent link="uarm_upper_arm_link"/>
       <child link="uarm_forearm_link"/>
-	  <axis xyz="0 0 1" />
+	  <axis xyz="1 0 0" />
 	  <limit lower="${joint_lower_limit}" upper="${joint_upper_limit}" effort="${joint_effort}" velocity="${joint_velocity}" />
     </joint>

Commit message: changed model and angle calculation

File: uarm_description/urdf/uarm3.urdf.xacro (robot description, xacro)
@@ -32,10 +32,4 @@
             </material>
       </visual>
-      <collision>
-        <origin xyz="0 0 0" rpy="0 0 0"  />
-        <geometry>
-            <mesh filename="package://uarm_description/meshes/uarm_base.stl" scale="0.001 0.001 0.001"/>
-        </geometry>
-       </collision>
     </link>
     <joint name="base_body_j" type="revolute">
@@ -90,17 +84,22 @@
         </material>
       </visual>
-	  <collision>
-		<origin xyz="0 0 0" rpy="0 0 ${M_PI/2}" />
-		<geometry>
-			<mesh filename="package://uarm_description/meshes/uarm_upper_arm.stl" scale="0.001 0.001 0.001"/>
-        </geometry>
-	  </collision>
     </link>
-    <joint name="upper_arm_forearm_j" type="revolute">
-      <origin xyz="0 0.048 0.138 " rpy="${joint_forearm_offset} 0 0"/>
+    <joint name="mimic_joint_1" type="revolute">
+    <origin xyz="0 0.048 0.138" rpy="${joint_forearm_offset} 0 0"/>
       <parent link="uarm_upper_arm_link"/>
+      <child link="virtual_link_2"/>
+      <mimic joint="body_upper_arm_j" multiplier="-1"/>
+      <axis xyz="1 0 0"/>
+      <limit effort="200" velocity="1.9634" lower="-${M_PI}" upper="${M_PI}"/>
+    </joint>
+    <link name="virtual_link_2">
+    </link>
+    <joint name="mimic_joint_2" type="revolute">
+    <origin xyz="0 0 0" rpy="0 0 0"/>
+      <parent link="virtual_link_2"/>
       <child link="uarm_forearm_link"/>
-	  <axis xyz="1 0 0" />
-	  <limit lower="${joint_lower_limit}" upper="${joint_upper_limit}" effort="${joint_effort}" velocity="${joint_velocity}" />
+      <mimic joint="forearm_wrist_j" multiplier="-1"/>
+      <axis xyz="1 0 0"/>
+      <limit effort="200" velocity="1.9634" lower="-${M_PI}" upper="${M_PI}"/>
     </joint>
    <link name="uarm_forearm_link">
@@ -119,35 +118,10 @@
 		</material>
       </visual>
-	  <collision>
-		<origin xyz="0 0 0" rpy="0 0 ${M_PI/2}" />
-		<geometry>
-            <mesh filename="package://uarm_description/meshes/uarm_forearm.stl" scale="0.001 0.001 0.001"/>
-		</geometry>
-	  </collision>
    </link>
-<!--
-    <joint name="forearm_wrist_j" type="continuous">
-      <origin xyz="0 -0.145 -0.068" rpy="-2.8 0 0"/>
+    <joint name="forearm_wrist_j" type="revolute">
+      <origin xyz="0 -0.145 -0.068" rpy="${-joint_upper_arm_offset-joint_forearm_offset-1.58} 0 0"/>
       <parent link="uarm_forearm_link"/>
       <child link="uarm_wrist_link"/>
-    </joint>
--->
-    <joint name="mimic_joint_1" type="revolute">
-    <origin xyz="0 -0.145 -0.068" rpy="${-joint_upper_arm_offset-joint_forearm_offset-1.58} 0 0"/>
-      <parent link="uarm_forearm_link"/>
-      <child link="virtual_link_2"/>
-      <mimic joint="body_upper_arm_j" multiplier="-1"/>
-      <axis xyz="1 0 0"/>
-      <limit effort="200" velocity="1.9634" lower="-${M_PI}" upper="${M_PI}"/>
-    </joint>
-    <link name="virtual_link_2">
-    </link>
-    <joint name="mimic_joint_2" type="revolute">
-    <origin xyz="0 0 0" rpy="0 0 0"/>
-      <parent link="virtual_link_2"/>
-      <child link="uarm_wrist_link"/>
-      <mimic joint="upper_arm_forearm_j" multiplier="-1"/>
-      <axis xyz="1 0 0"/>
-      <limit effort="200" velocity="1.9634" lower="-${M_PI}" upper="${M_PI}"/>
+      <limit effort="200" velocity="1.9634" lower="-0.68" upper="0.95"/>
     </joint>
     <link name="uarm_wrist_link">
@@ -179,8 +153,17 @@
       </visual>
     </link>
+    <joint name="fingers_j" type="revolute">
+      <origin xyz="0 0 0 " rpy="0 0 0"/>
+      <parent link="uarm_palm_link"/>
+      <child link="virtual_link_3"/>
+      <limit effort="200" velocity="1.9634" lower="-1.134" upper="-0.349"/>
+    </joint>
+    <link name="virtual_link_3">
+    </link>
     <joint name="palm_left_finger_j" type="revolute">
       <origin xyz="0.035 -0.008 0 " rpy="0 ${M_PI/2} 0"/>
       <parent link="uarm_palm_link"/>
       <child link="uarm_left_finger_link"/>
+      <mimic joint="fingers_j" multiplier="-0.5" offset="${-0.349/2}"/>
       <limit effort="200" velocity="1.9634" lower="0" upper="0.40"/>
     </joint>
@@ -198,5 +181,5 @@
       <parent link="uarm_palm_link"/>
       <child link="uarm_right_finger_link"/>
-      <mimic joint="palm_left_finger_j" multiplier="-1"/>
+      <mimic joint="fingers_j" multiplier="0.5" offset="${0.349/2}"/>
       <limit effort="200" velocity="1.9634" lower="-0.4" upper="0"/>
     </joint>
@@ -210,15 +193,4 @@
       </visual>
     </link>
-<!--
-    <link name="uarm_left_finger_link">
-      <visual>
-        <origin xyz="0 0 0" rpy="0 0 0" />
-        <geometry>
-            <box size="0.001 0.001 0.001"/>
-        </geometry>
-        <material name="${color}" />
-      </visual>
-    </link>
--->
   </xacro:macro>
 </robot>

Commit message: changing model

File: uarm_description/urdf/uarm3.urdf.xacro (robot description, xacro)
@@ -8,6 +8,7 @@
     <xacro:property name="joint_effort" value="10000" />
     <xacro:property name="joint_velocity" value="100" />
-    <xacro:property name="joint_upper_arm_offset" value="-0.85"/>
-    <xacro:property name="joint_forearm_offset" value="-0.30" />
+    <xacro:property name="joint_upper_arm_visual_offset" value="-1.164696417"/>
+    <xacro:property name="joint_forearm_visual_offset" value="-0.475385253" />
+    <xacro:property name="joint_wrist_visual_offset" value="-0.290688836" />
  <!-- uArm description -->
   <xacro:macro name="uarm" params="parent  color *origin">
@@ -63,5 +64,5 @@
     </link>
     <joint name="body_upper_arm_j" type="revolute">
-      <origin xyz="0.069 0 0.021" rpy="${joint_upper_arm_offset} 0 ${-M_PI/2}"/>
+      <origin xyz="0.069 0 0.021" rpy="${joint_upper_arm_visual_offset} 0 ${-M_PI/2}"/>
       <parent link="uarm_body_link"/>
       <child link="uarm_upper_arm_link"/>
@@ -86,5 +87,5 @@
     </link>
     <joint name="mimic_joint_1" type="revolute">
-    <origin xyz="0 0.048 0.138" rpy="${joint_forearm_offset} 0 0"/>
+    <origin xyz="0 0.048 0.138" rpy="${joint_forearm_visual_offset} 0 0"/>
       <parent link="uarm_upper_arm_link"/>
       <child link="virtual_link_2"/>
@@ -120,5 +121,5 @@
    </link>
     <joint name="forearm_wrist_j" type="revolute">
-      <origin xyz="0 -0.145 -0.068" rpy="${-joint_upper_arm_offset-joint_forearm_offset-1.58} 0 0"/>
+      <origin xyz="0 -0.145 -0.068" rpy="${joint_wrist_visual_offset} 0 0"/>
       <parent link="uarm_forearm_link"/>
       <child link="uarm_wrist_link"/>

Commit message: model & angles calculation

File: uarm_description/urdf/uarm3.urdf.xacro (robot description, xacro)
@@ -8,7 +8,9 @@
     <xacro:property name="joint_effort" value="10000" />
     <xacro:property name="joint_velocity" value="100" />
-    <xacro:property name="joint_upper_arm_visual_offset" value="-1.164696417"/>
-    <xacro:property name="joint_forearm_visual_offset" value="-0.475385253" />
-    <xacro:property name="joint_wrist_visual_offset" value="-0.290688836" />
+    <xacro:property name="joint_left_visual_offset" value="0.35"/> <!-- "+" contr clock   -->
+    <xacro:property name="joint_right_visual_offset" value="-0.35" /> <!-- "-" contr clock   -->
+    <xacro:property name="joint_upper_arm_visual_offset" value="${-1.291+joint_left_visual_offset}"/> <!-- "+" contr clock   -->
+    <xacro:property name="joint_forearm_visual_offset" value="${-0.25-joint_left_visual_offset-joint_right_visual_offset}" /> <!-- "+" contr clock   -->
+    <xacro:property name="joint_wrist_visual_offset" value="${joint_right_visual_offset}" /> <!-- "+" contr clock   -->
  <!-- uArm description -->
   <xacro:macro name="uarm" params="parent  color *origin">
@@ -67,5 +69,5 @@
       <parent link="uarm_body_link"/>
       <child link="uarm_upper_arm_link"/>
-      <axis xyz="1 0 0" />
+      <axis xyz="-1 0 0" />
       <limit lower="${joint_lower_limit}" upper="${joint_upper_limit}" effort="${joint_effort}" velocity="${joint_velocity}" />
     </joint>
@@ -91,5 +93,5 @@
       <child link="virtual_link_2"/>
       <mimic joint="body_upper_arm_j" multiplier="-1"/>
-      <axis xyz="1 0 0"/>
+      <axis xyz="-1 0 0"/>
       <limit effort="200" velocity="1.9634" lower="-${M_PI}" upper="${M_PI}"/>
     </joint>
@@ -101,5 +103,5 @@
       <child link="uarm_forearm_link"/>
       <mimic joint="forearm_wrist_j" multiplier="-1"/>
-      <axis xyz="1 0 0"/>
+      <axis xyz="-1 0 0"/>
       <limit effort="200" velocity="1.9634" lower="-${M_PI}" upper="${M_PI}"/>
     </joint>
@@ -124,5 +126,6 @@
       <parent link="uarm_forearm_link"/>
       <child link="uarm_wrist_link"/>
-      <limit effort="200" velocity="1.9634" lower="-0.68" upper="0.95"/>
+      <axis xyz="-1 0 0"/>
+      <limit effort="200" velocity="1.9634" lower="-1.68" upper="0.95"/>
     </joint>
     <link name="uarm_wrist_link">
