Commit message: changed urdf model

File: uarm_description/urdf/robot.urdf.xacro (robot description, xacro)
@@ -3,5 +3,5 @@
   <!-- The following included files set up definitions of parts of the robot body -->
 <xacro:property name="M_PI" value="3.1415926535897931" />
-  <xacro:include filename="$(find uarm_description)/urdf/uarm.urdf.xacro" />
+  <xacro:include filename="$(find uarm_description)/urdf/uarm3.urdf.xacro" />
 <!--
   <xacro:include filename="$(find uarm_description)/urdf/camera.urdf.xacro" />

File: uarm_description/urdf/uarm3.urdf.xacro (robot description, xacro)
@@ -8,4 +8,6 @@
     <xacro:property name="joint_effort" value="10000" />
     <xacro:property name="joint_velocity" value="100" />
+    <xacro:property name="joint_upper_arm_offset" value="-0.85"/>
+    <xacro:property name="joint_forearm_offset" value="-0.30" />
  <!-- uArm description -->
   <xacro:macro name="uarm" params="parent  color *origin">
@@ -51,5 +53,5 @@
       </inertial>
       <visual>
-        <origin xyz="0 0 0" rpy="0 ${M_PI/2} 0" />
+       <origin xyz="0 0 0" rpy="0 ${M_PI/2} 0" />
         <geometry>
             <mesh filename="package://uarm_description/meshes/uarm_body.stl" scale="0.001 0.001 0.001"/>
@@ -60,12 +62,12 @@
 	  </visual>
 	  <collision>
-        <origin xyz="0 0 0" rpy="0 ${M_PI/2} 0" />
+        <origin xyz="0.032 0 0" rpy="0 ${M_PI/2} 0" />
 		<geometry>
-			 <mesh filename="package://uarm_description/meshes/uarm_body.stl" scale="0.001 0.001 0.001"/>
+			 <box size="0.1 0.1 0.035" />
 		</geometry>
       </collision>
     </link>
     <joint name="body_upper_arm_j" type="revolute">
-      <origin xyz="0.069 0 0.021" rpy="-3 0 ${-M_PI/2}"/>
+      <origin xyz="0.069 0 0.021" rpy="${joint_upper_arm_offset} 0 ${-M_PI/2}"/>
       <parent link="uarm_body_link"/>
       <child link="uarm_upper_arm_link"/>
@@ -96,5 +98,5 @@
     </link>
     <joint name="upper_arm_forearm_j" type="revolute">
-      <origin xyz="0 0.048 0.138 " rpy="1.052 0 0"/>
+      <origin xyz="0 0.048 0.138 " rpy="${joint_forearm_offset} 0 0"/>
       <parent link="uarm_upper_arm_link"/>
       <child link="uarm_forearm_link"/>
@@ -124,4 +126,5 @@
 	  </collision>
    </link>
+<!--
     <joint name="forearm_wrist_j" type="continuous">
       <origin xyz="0 -0.145 -0.068" rpy="-2.8 0 0"/>
@@ -129,4 +132,23 @@
       <child link="uarm_wrist_link"/>
     </joint>
+-->
+    <joint name="mimic_joint_1" type="revolute">
+    <origin xyz="0 -0.145 -0.068" rpy="${-joint_upper_arm_offset-joint_forearm_offset-1.58} 0 0"/>
+      <parent link="uarm_forearm_link"/>
+      <child link="virtual_link_2"/>
+      <mimic joint="body_upper_arm_j" multiplier="-1"/>
+      <axis xyz="1 0 0"/>
+      <limit effort="200" velocity="1.9634" lower="-${M_PI}" upper="${M_PI}"/>
+    </joint>
+    <link name="virtual_link_2">
+    </link>
+    <joint name="mimic_joint_2" type="revolute">
+    <origin xyz="0 0 0" rpy="0 0 0"/>
+      <parent link="virtual_link_2"/>
+      <child link="uarm_wrist_link"/>
+      <mimic joint="upper_arm_forearm_j" multiplier="-1"/>
+      <axis xyz="1 0 0"/>
+      <limit effort="200" velocity="1.9634" lower="-${M_PI}" upper="${M_PI}"/>
+    </joint>
     <link name="uarm_wrist_link">
       <visual>
@@ -140,8 +162,9 @@
       </visual>
     </link>
-    <joint name="wrist_palm_j" type="continuous">
+    <joint name="wrist_palm_j" type="revolute">
       <origin xyz="0.0022 -0.036 -0.011" rpy=" ${-M_PI/2} ${M_PI/2} 0"/>
       <parent link="uarm_wrist_link"/>
       <child link="uarm_palm_link"/>
+      <limit effort="200" velocity="1.9634" lower="-${M_PI/2}" upper="${M_PI/2}"/>
     </joint>
     <link name="uarm_palm_link">
@@ -156,8 +179,9 @@
       </visual>
     </link>
-    <joint name="palm_left_finger_j" type="continuous">
+    <joint name="palm_left_finger_j" type="revolute">
       <origin xyz="0.035 -0.008 0 " rpy="0 ${M_PI/2} 0"/>
       <parent link="uarm_palm_link"/>
       <child link="uarm_left_finger_link"/>
+      <limit effort="200" velocity="1.9634" lower="0" upper="0.40"/>
     </joint>
     <link name="uarm_left_finger_link">
@@ -170,8 +194,10 @@
       </visual>
     </link>
-    <joint name="palm_right_finger_j" type="continuous">
+    <joint name="palm_right_finger_j" type="revolute">
       <origin xyz="0.035 0.008 0" rpy="0 ${M_PI/2} 0"/>
       <parent link="uarm_palm_link"/>
       <child link="uarm_right_finger_link"/>
+      <mimic joint="palm_left_finger_j" multiplier="-1"/>
+      <limit effort="200" velocity="1.9634" lower="-0.4" upper="0"/>
     </joint>
     <link name="uarm_right_finger_link">

Commit message: clear code

File: uarm_description/urdf/robot.urdf.xacro (robot description, xacro)
@@ -3,5 +3,5 @@
   <!-- The following included files set up definitions of parts of the robot body -->
 <xacro:property name="M_PI" value="3.1415926535897931" />
-  <xacro:include filename="$(find uarm_description)/urdf/uarm3.urdf.xacro" />
+  <xacro:include filename="$(find uarm_description)/urdf/uarm.urdf.xacro" />
 <!--
   <xacro:include filename="$(find uarm_description)/urdf/camera.urdf.xacro" />

File: uarm_description/urdf/uarm.urdf.xacro (robot description, xacro)
@@ -1,4 +1,16 @@
 <?xml version="1.0"?>
 <robot xmlns:xacro="http://www.ros.org/wiki/xacro">
+<!-- Pi parameter -->
+    <xacro:property name="pi" value="3.1415926535897931" />
+<!-- Joint properties -->
+    <xacro:property name="joint_lower_limit" value="-${1.5}" />
+    <xacro:property name="joint_upper_limit" value="${1.5}" />
+    <xacro:property name="joint_effort" value="10000" />
+    <xacro:property name="joint_velocity" value="100" />
+    <xacro:property name="joint_left_visual_offset" value="0.35"/> <!-- "+" contr clock   -->
+    <xacro:property name="joint_right_visual_offset" value="-0.35" /> <!-- "-" contr clock   -->
+    <xacro:property name="joint_upper_arm_visual_offset" value="${-1.291+joint_left_visual_offset}"/> <!-- "+" contr clock   -->
+    <xacro:property name="joint_forearm_visual_offset" value="${-0.25-joint_left_visual_offset-joint_right_visual_offset}" /> <!-- "+" contr clock   -->
+    <xacro:property name="joint_wrist_visual_offset" value="${joint_right_visual_offset}" /> <!-- "+" contr clock   -->
  <!-- uArm description -->
   <xacro:macro name="uarm" params="parent  color *origin">
@@ -9,4 +21,9 @@
     </joint>
     <link name="uarm_base_link">
+      <inertial>
+        <origin xyz="0 0 0" />
+        <mass value="0.01"/>
+        <inertia  ixx="0.01" ixy="0" ixz="0" iyy="0.01" iyz="0" izz="0.01"/>
+      </inertial>
       <visual>
         <origin xyz="0 0 0" rpy="0 0 0" />
@@ -14,41 +31,85 @@
             <mesh filename="package://uarm_description/meshes/uarm_base.stl" scale="0.001 0.001 0.001"/>
         </geometry>
-        <material name="${color}" />
-      </visual>
-    </link>
-    <joint name="base_body_j" type="continuous">
+            <material name="grey">
+                <color rgba="0.5 0.5 0.5 1" />
+            </material>
+      </visual>
+    </link>
+    <joint name="base_body_j" type="revolute">
       <origin xyz="0 0 0" rpy="0 ${-M_PI/2} 0"/>
       <parent link="uarm_base_link"/>
       <child link="uarm_body_link"/>
+      <axis xyz="1 0 0" />
+      <limit lower="${joint_lower_limit}" upper="${joint_upper_limit}" effort="${joint_effort}" velocity="${joint_velocity}" />
     </joint>
     <link name="uarm_body_link">
-      <visual>
-        <origin xyz="0 0 0" rpy="0 ${M_PI/2} 0" />
+	  <inertial>
+          <origin xyz="0 0 0" rpy="0 ${M_PI/2} 0" />
+          <mass value="0.01"/>
+          <inertia 	ixx="0.01" ixy="0" ixz="0" iyy="0.01" iyz="0" izz="0.01"/>
+      </inertial>
+      <visual>
+       <origin xyz="0 0 0" rpy="0 ${M_PI/2} 0" />
         <geometry>
             <mesh filename="package://uarm_description/meshes/uarm_body.stl" scale="0.001 0.001 0.001"/>
         </geometry>
-        <material name="${color}" />
-      </visual>
-    </link>
-    <joint name="body_upper_arm_j" type="continuous">
-      <origin xyz="0.069 0 0.021" rpy="-3 0 ${-M_PI/2}"/>
+            <material name="">
+                 <color rgba="0.7 0.7 0 1" />
+            </material>
+	  </visual>
+	  <collision>
+        <origin xyz="0.032 0 0" rpy="0 ${M_PI/2} 0" />
+		<geometry>
+			 <box size="0.1 0.1 0.035" />
+		</geometry>
+      </collision>
+    </link>
+    <joint name="body_upper_arm_j" type="revolute">
+      <origin xyz="0.069 0 0.021" rpy="${joint_upper_arm_visual_offset} 0 ${-M_PI/2}"/>
       <parent link="uarm_body_link"/>
       <child link="uarm_upper_arm_link"/>
+      <axis xyz="-1 0 0" />
+      <limit lower="${joint_lower_limit}" upper="${joint_upper_limit}" effort="${joint_effort}" velocity="${joint_velocity}" />
     </joint>
     <link name="uarm_upper_arm_link">
-      <visual>
-        <origin xyz="0 0 ${0}" rpy="0 0 ${M_PI/2}" />
+       <inertial>
+         <origin xyz="0 0 0" rpy="0 0 ${M_PI/2}" />
+         <mass value="0.01"/>
+         <inertia 	ixx="0.01" ixy="0" ixz="0" iyy="0.01" iyz="0" izz="0.01"/>
+       </inertial>
+      <visual>
+        <origin xyz="0 0 0" rpy="0 0 ${M_PI/2}" />
         <geometry>
             <mesh filename="package://uarm_description/meshes/uarm_upper_arm.stl" scale="0.001 0.001 0.001"/>
         </geometry>
-        <material name="${color}" />
-      </visual>
-    </link>
-    <joint name="upper_arm_forearm_j" type="continuous">
-      <origin xyz="0 0.048 0.138 " rpy="1.052 0 0"/>
+        <material name="">
+            <color rgba="0 0.7 0.7 1" />
+        </material>
+      </visual>
+    </link>
+    <joint name="mimic_joint_1" type="revolute">
+    <origin xyz="0 0.048 0.138" rpy="${joint_forearm_visual_offset} 0 0"/>
       <parent link="uarm_upper_arm_link"/>
+      <child link="virtual_link_2"/>
+      <mimic joint="body_upper_arm_j" multiplier="-1"/>
+      <axis xyz="-1 0 0"/>
+      <limit effort="200" velocity="1.9634" lower="-${M_PI}" upper="${M_PI}"/>
+    </joint>
+    <link name="virtual_link_2">
+    </link>
+    <joint name="mimic_joint_2" type="revolute">
+    <origin xyz="0 0 0" rpy="0 0 0"/>
+      <parent link="virtual_link_2"/>
       <child link="uarm_forearm_link"/>
+      <mimic joint="forearm_wrist_j" multiplier="-1"/>
+      <axis xyz="-1 0 0"/>
+      <limit effort="200" velocity="1.9634" lower="-${M_PI}" upper="${M_PI}"/>
     </joint>
    <link name="uarm_forearm_link">
+	  <inertial>
+		<origin xyz="0 0 0" rpy="0 0 ${M_PI/2}" />
+		<mass value="0.01"/>
+		<inertia 	ixx="0.01" ixy="0" ixz="0" iyy="0.01" iyz="0" izz="0.01"/>
+	  </inertial>
       <visual>
         <origin xyz="0 0 0" rpy="0 0 ${M_PI/2}" />
@@ -56,11 +117,15 @@
             <mesh filename="package://uarm_description/meshes/uarm_forearm.stl" scale="0.001 0.001 0.001"/>
         </geometry>
-        <material name="${color}" />
-      </visual>
-    </link>
-    <joint name="forearm_wrist_j" type="continuous">
-      <origin xyz="0 -0.145 -0.068" rpy="-2.8 0 0"/>
+		<material name="">
+			<color rgba="0.7 0 0.7 1" />
+		</material>
+      </visual>
+   </link>
+    <joint name="forearm_wrist_j" type="revolute">
+      <origin xyz="0 -0.145 -0.068" rpy="${joint_wrist_visual_offset} 0 0"/>
       <parent link="uarm_forearm_link"/>
       <child link="uarm_wrist_link"/>
+      <axis xyz="-1 0 0"/>
+      <limit effort="200" velocity="1.9634" lower="-1.68" upper="0.95"/>
     </joint>
     <link name="uarm_wrist_link">
@@ -70,11 +135,14 @@
             <mesh filename="package://uarm_description/meshes/uarm_wrist.stl" scale="0.001 0.001 0.001"/>
         </geometry>
-        <material name="${color}" />
-      </visual>
-    </link>
-    <joint name="wrist_palm_j" type="continuous">
+        <material name="">
+			<color rgba="0.5 0 0.7 1" />
+		</material>
+      </visual>
+    </link>
+    <joint name="wrist_palm_j" type="revolute">
       <origin xyz="0.0022 -0.036 -0.011" rpy=" ${-M_PI/2} ${M_PI/2} 0"/>
       <parent link="uarm_wrist_link"/>
       <child link="uarm_palm_link"/>
+      <limit effort="200" velocity="1.9634" lower="-${M_PI/2}" upper="${M_PI/2}"/>
     </joint>
     <link name="uarm_palm_link">
@@ -84,11 +152,23 @@
             <mesh filename="package://uarm_description/meshes/uarm_palm.stl" scale="0.001 0.001 0.001"/>
         </geometry>
-        <material name="${color}" />
-      </visual>
-    </link>
-    <joint name="palm_left_finger_j" type="continuous">
+        <material name="">
+			<color rgba="0.7 0 0.5 1" />
+		</material>
+      </visual>
+    </link>
+    <joint name="fingers_j" type="revolute">
+      <origin xyz="0 0 0 " rpy="0 0 0"/>
+      <parent link="uarm_palm_link"/>
+      <child link="virtual_link_3"/>
+      <limit effort="200" velocity="1.9634" lower="-1.134" upper="-0.349"/>
+    </joint>
+    <link name="virtual_link_3">
+    </link>
+    <joint name="palm_left_finger_j" type="revolute">
       <origin xyz="0.035 -0.008 0 " rpy="0 ${M_PI/2} 0"/>
       <parent link="uarm_palm_link"/>
       <child link="uarm_left_finger_link"/>
+      <mimic joint="fingers_j" multiplier="-0.5" offset="${-0.349/2}"/>
+      <limit effort="200" velocity="1.9634" lower="0" upper="0.40"/>
     </joint>
     <link name="uarm_left_finger_link">
@@ -101,8 +181,10 @@
       </visual>
     </link>
-    <joint name="palm_right_finger_j" type="continuous">
+    <joint name="palm_right_finger_j" type="revolute">
       <origin xyz="0.035 0.008 0" rpy="0 ${M_PI/2} 0"/>
       <parent link="uarm_palm_link"/>
       <child link="uarm_right_finger_link"/>
+      <mimic joint="fingers_j" multiplier="0.5" offset="${0.349/2}"/>
+      <limit effort="200" velocity="1.9634" lower="-0.4" upper="0"/>
     </joint>
     <link name="uarm_right_finger_link">
@@ -115,15 +197,4 @@
       </visual>
     </link>
-<!--
-    <link name="uarm_left_finger_link">
-      <visual>
-        <origin xyz="0 0 0" rpy="0 0 0" />
-        <geometry>
-            <box size="0.001 0.001 0.001"/>
-        </geometry>
-        <material name="${color}" />
-      </visual>
-    </link>
--->
   </xacro:macro>
 </robot>
